File: FullSchematic/AmplifierSchematic_20230805.kicad_sch (KiCad schematic)
At the start: 36 parts, among them U1 IR2181STRPBF, U2 IR2181STRPBF, U3 IPB009N03L G, U4 IPB009N03L G, U5 IPB009N03L G, U6 IPB009N03L G

Commit message: Schematic/Footprint Update
Corrected Footprint / Schematic for PCB Design and Changed 10k Resistors to 0603 size.
Connections:
- net +12V: no longer U3.4 (Drain), U5.4 (Drain)
- net at C10.2, L2.1, U2.6 (VS)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: no longer U6.4 (Drain)
- net at C9.2, L1.1, U1.6 (VS)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: no longer U4.4 (Drain)
Changed lines of the file:
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@@
   (junction (at 109.982 116.84) (diameter 0) (color 0 0 0 0)
   )
-  (junction (at 156.21 27.686) (diameter 0) (color 0 0 0 0)
-  )
   (junction (at 136.652 148.844) (diameter 0) (color 0 0 0 0)
   )
   (junction (at 103.378 40.132) (diameter 0) (color 0 0 0 0)
   )
-  (junction (at 156.21 61.976) (diameter 0) (color 0 0 0 0)
-  )
   (junction (at 109.982 56.896) (diameter 0) (color 0 0 0 0)
   )
@@
   (junction (at 198.374 150.622) (diameter 0) (color 0 0 0 0)
   )
-  (junction (at 156.21 104.394) (diameter 0) (color 0 0 0 0)
-  )
   (junction (at 53.594 131.064) (diameter 0) (color 0 0 0 0)
   )
@@
   (junction (at 163.83 127.508) (diameter 0) (color 0 0 0 0)
   )
-  (junction (at 156.21 138.684) (diameter 0) (color 0 0 0 0)
-  )
   (junction (at 158.75 86.106) (diameter 0) (color 0 0 0 0)
   )
@@
     (stroke (width 0) (type default))
   )
-  (wire (pts (xy 156.21 96.774) (xy 156.21 104.394))
+  (wire (pts (xy 156.21 96.774) (xy 156.21 107.188))
     (stroke (width 0) (type default))
   )
@@
     (stroke (width 0) (type default))
   )
-  (wire (pts (xy 161.29 61.976) (xy 161.29 63.5))
-    (stroke (width 0) (type default))
-  )
   (wire (pts (xy 163.83 79.756) (xy 163.83 86.106))
     (stroke (width 0) (type default))
   )
-  (wire (pts (xy 161.29 27.686) (xy 161.29 30.48))
-    (stroke (width 0) (type default))
-  )
   (wire (pts (xy 136.906 72.136) (xy 139.7 72.136))
     (stroke (width 0) (type default))
@@
     (stroke (width 0) (type default))
   )
-  (wire (pts (xy 161.29 104.394) (xy 161.29 107.188))
-    (stroke (width 0) (type default))
-  )
   (wire (pts (xy 64.516 56.896) (xy 72.644 56.896))
     (stroke (width 0) (type default))
@@
     (stroke (width 0) (type default))
   )
-  (wire (pts (xy 156.21 20.066) (xy 156.21 27.686))
-    (stroke (width 0) (type default))
-  )
   (wire (pts (xy 43.688 128.524) (xy 72.644 128.524))
     (stroke (width 0) (type default))
@@
     (stroke (width 0) (type default))
   )
-  (wire (pts (xy 156.21 61.976) (xy 156.21 63.5))
+  (wire (pts (xy 156.21 56.896) (xy 156.21 63.5))
     (stroke (width 0) (type default))
   )
@@
     (stroke (width 0) (type default))
   )
-  (wire (pts (xy 156.21 133.604) (xy 156.21 138.684))
+  (wire (pts (xy 156.21 133.604) (xy 156.21 140.208))
     (stroke (width 0) (type default))
   )
@@
     (stroke (width 0) (type default))
   )
-  (wire (pts (xy 156.21 61.976) (xy 161.29 61.976))
-    (stroke (width 0) (type default))
-  )
   (wire (pts (xy 120.904 115.824) (xy 125.73 115.824))
     (stroke (width 0) (type default))
@@
     (stroke (width 0) (type default))
   )
-  (wire (pts (xy 156.21 138.684) (xy 161.29 138.684))
-    (stroke (width 0) (type default))
-  )
   (wire (pts (xy 40.386 54.356) (xy 54.356 54.356))
     (stroke (width 0) (type default))
@@
     (stroke (width 0) (type default))
   )
-  (wire (pts (xy 156.21 104.394) (xy 161.29 104.394))
-    (stroke (width 0) (type default))
-  )
   (wire (pts (xy 102.616 128.524) (xy 120.904 128.524))
     (stroke (width 0) (type default))
@@
     (stroke (width 0) (type default))
   )
-  (wire (pts (xy 156.21 56.896) (xy 156.21 61.976))
-    (stroke (width 0) (type default))
-  )
   (wire (pts (xy 148.59 123.444) (xy 148.59 127.508))
     (stroke (width 0) (type default))
@@
     (stroke (width 0) (type default))
   )
-  (wire (pts (xy 161.29 138.684) (xy 161.29 140.208))
-    (stroke (width 0) (type default))
-  )
   (wire (pts (xy 102.616 56.896) (xy 104.648 56.896))
     (stroke (width 0) (type default))
@@
     (stroke (width 0) (type default))
   )
-  (wire (pts (xy 156.21 27.686) (xy 161.29 27.686))
-    (stroke (width 0) (type default))
-  )
   (wire (pts (xy 109.982 20.066) (xy 109.982 29.21))
     (stroke (width 0) (type default))
@@
     (stroke (width 0) (type default))
   )
-  (wire (pts (xy 156.21 104.394) (xy 156.21 107.188))
-    (stroke (width 0) (type default))
-  )
   (wire (pts (xy 109.982 50.546) (xy 109.982 56.896))
     (stroke (width 0) (type default))
@@
     (stroke (width 0) (type default))
   )
-  (wire (pts (xy 156.21 138.684) (xy 156.21 140.208))
-    (stroke (width 0) (type default))
-  )
   (wire (pts (xy 109.982 127.254) (xy 109.982 133.604))
     (stroke (width 0) (type default))
@@
     (stroke (width 0) (type default))
   )
-  (wire (pts (xy 156.21 27.686) (xy 156.21 30.48))
+  (wire (pts (xy 156.21 20.066) (xy 156.21 30.48))
     (stroke (width 0) (type default))
   )
@@
     (pin "6")
     (pin "7")
-    (pin "4")
     (pin "TAB")
     (instances
@@
     (pin "6")
     (pin "7")
-    (pin "4")
     (pin "TAB")
     (instances
@@
     (pin "6")
     (pin "7")
-    (pin "4")
     (pin "TAB")
     (instances
@@
     (pin "6")
     (pin "7")
-    (pin "4")
     (pin "TAB")
     (instances

Commit message: PCB V.1
Parts:
- removed TP1, TP3: TestPoint, TestPoint:TestPoint_2Pads_Pitch2.54mm_Drill0.8mm, symbol Connector:TestPoint
Changed lines of the file:
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@@
   (junction (at 148.59 133.604) (diameter 0) (color 0 0 0 0)
   )
-  (junction (at 43.688 128.524) (diameter 0) (color 0 0 0 0)
-  )
   (junction (at 136.906 72.136) (diameter 0) (color 0 0 0 0)
   )
@@
   (junction (at 198.374 150.622) (diameter 0) (color 0 0 0 0)
   )
-  (junction (at 53.594 131.064) (diameter 0) (color 0 0 0 0)
-  )
   (junction (at 64.516 42.164) (diameter 0) (color 0 0 0 0)
   )
@@
     (stroke (width 0) (type default))
   )
-  (wire (pts (xy 53.594 126.746) (xy 53.594 131.064))
-    (stroke (width 0) (type default))
-  )
   (wire (pts (xy 198.374 73.914) (xy 210.058 73.914))
     (stroke (width 0) (type default))
@@
     (stroke (width 0) (type default))
   )
-  (wire (pts (xy 43.688 128.524) (xy 72.644 128.524))
+  (wire (pts (xy 40.894 128.524) (xy 72.644 128.524))
     (stroke (width 0) (type default))
   )
@@
     (stroke (width 0) (type default))
   )
-  (wire (pts (xy 43.688 126.746) (xy 43.688 128.524))
-    (stroke (width 0) (type default))
-  )
   (wire (pts (xy 163.83 46.736) (xy 163.83 50.8))
     (stroke (width 0) (type default))
@@
     (stroke (width 0) (type default))
   )
-  (wire (pts (xy 40.894 128.524) (xy 43.688 128.524))
-    (stroke (width 0) (type default))
-  )
   (wire (pts (xy 109.982 56.896) (xy 148.59 56.896))
     (stroke (width 0) (type default))
@@
     (stroke (width 0) (type default))
   )
-  (wire (pts (xy 40.894 131.064) (xy 53.594 131.064))
-    (stroke (width 0) (type default))
-  )
   (wire (pts (xy 54.356 54.356) (xy 72.644 54.356))
     (stroke (width 0) (type default))
@@
     (stroke (width 0) (type default))
   )
-  (wire (pts (xy 53.594 131.064) (xy 72.644 131.064))
+  (wire (pts (xy 40.894 131.064) (xy 72.644 131.064))
     (stroke (width 0) (type default))
   )
@@
         (path "/6d92e519-f2b8-4f1a-b6f2-abd18cbdca99"
           (reference "U6") (unit 1)
-        )
-      )
-    )
-  )
-  (symbol (lib_id "Connector:TestPoint") (at 53.594 126.746 0) (unit 1)
-    (in_bom yes) (on_board yes) (dnp no)
-    (property "Reference" "TP3" (at 49.276 118.11 0)
-      (effects (font (size 1.27 1.27)) (justify left))
-    )
-    (property "Value" "TestPoint" (at 49.276 120.65 0)
-      (effects (font (size 1.27 1.27)) (justify left))
-    )
-    (property "Footprint" "TestPoint:TestPoint_2Pads_Pitch2.54mm_Drill0.8mm" (at 58.674 126.746 0)
-      (effects (font (size 1.27 1.27)) hide)
-    )
-    (property "Datasheet" "~" (at 58.674 126.746 0)
-      (effects (font (size 1.27 1.27)) hide)
-    )
-    (pin "1")
-    (instances
-      (project "FullSchematic"
-        (path "/650f0e66-3493-4c97-9577-99f99fcd23df/f9f03856-6747-4585-ae8a-ad2bb4f2bff9"
-          (reference "TP3") (unit 1)
-        )
-      )
-      (project "AmplifierSchematic_4_8_2023"
-        (path "/6d92e519-f2b8-4f1a-b6f2-abd18cbdca99"
-          (reference "TP6") (unit 1)
         )
       )
@@
         )
       )
-    )
-  )
-  (symbol (lib_id "Connector:TestPoint") (at 43.688 126.746 0) (unit 1)
-    (in_bom yes) (on_board yes) (dnp no)
-    (property "Reference" "TP1" (at 39.37 118.11 0)
-      (effects (font (size 1.27 1.27)) (justify left))
-    )
-    (property "Value" "TestPoint" (at 39.37 120.65 0)
-      (effects (font (size 1.27 1.27)) (justify left))
-    )
-    (property "Footprint" "TestPoint:TestPoint_2Pads_Pitch2.54mm_Drill0.8mm" (at 48.768 126.746 0)
-      (effects (font (size 1.27 1.27)) hide)
-    )
-    (property "Datasheet" "~" (at 48.768 126.746 0)
-      (effects (font (size 1.27 1.27)) hide)
-    )
-    (pin "1")
-    (instances
-      (project "FullSchematic"
-        (path "/650f0e66-3493-4c97-9577-99f99fcd23df/f9f03856-6747-4585-ae8a-ad2bb4f2bff9"
-          (reference "TP1") (unit 1)
-        )
-      )
-      (project "AmplifierSchematic_4_8_2023"
-        (path "/6d92e519-f2b8-4f1a-b6f2-abd18cbdca99"
-          (reference "TP5") (unit 1)
-        )
-      )

Commit message: Added silkscreen diodes for real
Parts:
- added D3, D4: MURS320T3G, Diode_SMD:D_SMC, symbol Device:D
- renumbered TP2 to TP1, TP4 to TP2, TP5 to TP3, TP6 to TP4, TP7 to TP5, TP8 to TP6
Connections:
- net +12V: now also D3.1 (K), D4.1 (K)
- net at C10.2, L2.1, U2.6 (VS)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: now also D4.2 (A)
- net at C9.2, L1.1, U1.6 (VS)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: now also D3.2 (A)
Other:
- moved on the sheet: C11, C12
